File: EGA2RGBC_EPROM/EGA2RGBC.kicad_pcb (KiCad board)
At the start: 2 copper layers, 59.7 x 45.1 mm, 23 parts, among them J1 EGA Input, J3 CSync Selection, J4 Power, J5 Video Out, U1 27C010, U2 74LS244

Commit message: Add new revision of board
Parts:
- added C1: 22pF, Capacitor_THT:C_Disc_D3.0mm_W2.0mm_P2.50mm, F.Cu at (140.4, 72.4)
- added C2: 22pF, Capacitor_THT:C_Disc_D3.0mm_W2.0mm_P2.50mm, F.Cu at (130.2, 72.4)
- added C3: 22pF, Capacitor_THT:C_Disc_D3.0mm_W2.0mm_P2.50mm, F.Cu at (120.0, 72.4)
- added RN1: 10k, Resistor_THT:R_Array_SIP9, F.Cu at (99.7, 45.1)
- R3, R5, R7: value 1.5k -> 680
- moved R2 2.54 mm to (137.8, 69.8)
- moved R3 2.54 mm to (137.8, 67.3)
- moved J1 2.01 mm to (102.2, 40.0)
Routing:
- net VCC: track 135.6 -> 118.4 mm
- net /DEC_B: track 55.2 -> 38.7 mm
- net GND: track 185.7 -> 172.7 mm
- net /IN_B_I: track 11.2 -> 23.5 mm
- net /IN_VS: track 15.8 -> 28.2 mm
- net /MODE_IN: track 28.5 -> 17.3 mm
- net /OUT_G_I: track 47.4 -> 37.3 mm
- net /IN_G: track 7.64 -> 16.2 mm
- net /IN_R: track 13.8 -> 19.4 mm
- net /OUT_R: track 40.1 -> 34.6 mm
- net /IN_HS: track 33.0 -> 38.5 mm
- net /OUT_G: track 32.8 -> 37.7 mm, vias 1 -> 0
- net /IN_B: track 14.6 -> 19.4 mm
- net /DEC_B_I: track 30.1 -> 34.7 mm
- net /ANALOG_B: track 16.1 -> 20.4 mm
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Other:
- board text added: "rev 1.2"
- board text removed: "rev 1.1"
